Commit message: keep balance without move arm

File: resources/robots/WF_TRON1A/urdf/robot_with_arm.urdf (robot description, URDF)
Before this commit: robot wheel_biped, 10 links, 9 joints
Links:
- added link airbot_arm, mass 0.77705; visual mesh filename=../meshes/airbot_arm.STL
- added link airbot_arm_base, mass 0.17; visual box size=0.15 0.15 0.006
- added link link1, mass 0.5571; visual mesh filename=../meshes/link1.STL
- added link link2, mass 0.64621; collision box size=0.2 0.04 0.04; visual mesh filename=../meshes/link2.STL
- added link link3, mass 0.28804; collision box size=0.04 0.35 0.04; visual mesh filename=../meshes/link3.STL
- added link link4, mass 0.34876; visual mesh filename=../meshes/link4.STL
- added link link5, mass 0.36132; visual mesh filename=../meshes/link5.STL
- added link link6, mass 0.65361; collision box size=0.08 0.04 0.1; visual mesh filename=../meshes/link6.STL
- link abad_L_Link: mass 1.469 -> 1.496
- link abad_R_Link: mass 1.469 -> 1.496
- link base_Link: geometry collision box size=0.25 0.26 0.14; visual mesh filename=../meshes/base_Link.STL
- link wheel_L_Link: geometry collision cylinder length=0.017 radius=0.127; visual mesh filename=../meshes/wheel_L_Link.STL
- link wheel_R_Link: geometry collision cylinder length=0.017 radius=0.127; visual mesh filename=../meshes/wheel_R_Link.STL
Joints:
- added joint J1: type revolute, parent airbot_arm, child link1, origin xyz=0 0 0.1172 rpy=0 0 0, axis 0 0 1, limit lower=-3.14 upper=2.09 effort=18 velocity=3.14
- added joint J2: type revolute, parent link1, child link2, origin xyz=0 0 0 rpy=1.5708 -2.7549 0, axis 0 0 1, limit lower=-2.96 upper=0.17 effort=18 velocity=3.14
- added joint J3: type revolute, parent link2, child link3, origin xyz=0.27009 0 0 rpy=0 0 1.9575, axis 0 0 1, limit lower=-0.087 upper=3.14 effort=18 velocity=3.14
- added joint J4: type revolute, parent link3, child link4, origin xyz=0 0.30854 0 rpy=-1.5708 -1.5708 0, axis 0 0 1, limit lower=-2.96 upper=2.96 effort=3 velocity=6.28
- added joint J5: type revolute, parent link4, child link5, origin xyz=0 0 0 rpy=1.5708 0 0, axis 0 0 1, limit lower=-1.74 upper=1.74 effort=3 velocity=6.28
- added joint J6: type revolute, parent link5, child link6, origin xyz=0 0.26145 0 rpy=-1.5708 0 0, axis 0 0 1, limit lower=-3.14 upper=3.14 effort=3 velocity=6.28
- added joint airbot_arm_base_joint: type fixed, parent base_Link, child airbot_arm_base, origin xyz=0.00166 0 0.0195 rpy=0. 0. 0.
- added joint airbot_arm_joint: type fixed, parent airbot_arm_base, child airbot_arm, origin xyz=0.0245 0. 0.003 rpy=0. 0. 0.
- joint abad_L_Joint: limit lower=-0.38397 upper=1.39626 effort=80.0 velocity=15.0 -> lower=-0.38397 upper=1.39626 effort=80.0 velocity=20.0
- joint abad_R_Joint: limit lower=-1.39626 upper=0.38397 effort=80.0 velocity=15.0 -> lower=-1.39626 upper=0.38397 effort=80.0 velocity=20.0
- joint hip_L_Joint: limit lower=-1.012291 upper=1.396263 effort=80.0 velocity=15.0 -> lower=-1.012291 upper=1.396263 effort=80.0 velocity=20.0
- joint hip_R_Joint: limit lower=-1.396263 upper=1.012291 effort=80.0 velocity=15.0 -> lower=-1.396263 upper=1.012291 effort=80.0 velocity=20.0
- joint knee_L_Joint: limit lower=-0.872665 upper=1.361357 effort=80 velocity=15 -> lower=-0.872665 upper=1.361357 effort=80 velocity=20
- joint knee_R_Joint: limit lower=-1.361357 upper=0.872665 effort=80 velocity=15 -> lower=-1.361357 upper=0.872665 effort=80 velocity=20
- joint wheel_L_Joint: limit lower=-1000000 upper=1000000 effort=40 velocity=40 -> lower=-100000 upper=100000 effort=40 velocity=40
- joint wheel_R_Joint: limit lower=-1000000 upper=1000000 effort=40 velocity=40 -> lower=-100000 upper=100000 effort=40 velocity=40
